File: ledDriver_cc/led_driver_cc_v2/led_driver_cc_v2.kicad_sch (KiCad schematic)
At the start: 25 parts, among them J1 Conn_01x08_Pin, J3 Conn_01x02_Female, U1 TSR_1-2490, U2 WeMos_D1_mini, U7 LM3404

Commit message: add partslib
Parts:
- removed U2: WeMos_D1_mini, Module:WEMOS_D1_mini_light, symbol MCU_Module:WeMos_D1_mini
- removed U7: LM3404, Package_SO:SOIC-8_3.9x4.9mm_P1.27mm, symbol LM3404:LM3404
- added ESP32_S1: ~, custom_footprints:ESP32-S3-Zero, symbol custom_symbols:ESP32_S3_Mini_Zero
- added U2: LM3404, Package_SO:SOIC-8_3.9x4.9mm_P1.27mm, symbol custom_symbols:LM3404
Connections:
- net +5V: now also C3.1, C5.1, U1.3 (Vout), ESP32_S1.1 (5V)
- net GND: now also ESP32_S1.2 (GND), U2.4 (GND)
- net PWM1: now also ESP32_S1.16 (GP13)
- net PWM2: now also ESP32_S1.15 (GP12)
- net PWM3: now also ESP32_S1.14 (GP11), U2.3 (DIM)
- net PWM4: now also ESP32_S1.13 (GP10)
- net VCC: now also U2.8 (VIN); no longer C3.1, C5.1, U1.3 (Vout)
- net at C14.1: now also U2.2 (BOOT)
- net at C14.2, D2.1 (K), L2.1: now also U2.1 (SW)
- net at C1.1: now also U2.7 (VCC)
- net at R19.1: now also U2.6 (RON)
Other:
- moved on the sheet: C1, C14, D2, J1, L2, R19, R3

Commit message: more custom parts
Parts:
- F1: footprint Fuse:Fuseholder_Littelfuse_Nano2_154x -> custom_footprints:Fuse_Littelfuse-NANO2-451_453
- L2: footprint Inductor_SMD:L_10.4x10.4_H4.8 -> Inductor_SMD:L_TDK_SLF10145
Changed lines of the file:
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@@
 			)
 		)
-		(property "Footprint" "Inductor_SMD:L_10.4x10.4_H4.8"
+		(property "Footprint" "Inductor_SMD:L_TDK_SLF10145"
 			(at 270.51 135.89 0)
 			(effects
@@
 			)
 		)
-		(property "Footprint" "Fuse:Fuseholder_Littelfuse_Nano2_154x"
+		(property "Footprint" "custom_footprints:Fuse_Littelfuse-NANO2-451_453"
 			(at 54.61 204.978 90)
 			(effects
