File: ledDriver_cc/led_driver_cc_v2/_autosave-led_driver_cc_v2.kicad_sch (KiCad schematic)
At the start: 25 parts, among them J1 Conn_01x08_Pin, J3 Conn_01x02_Female, U1 TSR_1-2490, U2 LM3404

Commit message: removed lib
Parts:
- added C15: 1uF, Capacitor_SMD:C_1206_3216Metric_Pad1.33x1.80mm_HandSolder, symbol Device:C
- added C16: 100nF, Capacitor_SMD:C_1206_3216Metric_Pad1.33x1.80mm_HandSolder, symbol Device:C
- added C18: 10uF, Capacitor_SMD:C_1210_3225Metric_Pad1.33x2.70mm_HandSolder, symbol Device:C
- C1: value C -> 100n
- C14: value C -> 10nF
- C2: footprint Capacitor_THT:CP_Radial_D13.0mm_P5.00mm -> Capacitor_SMD:CP_Elec_10x10
- R3: value R -> 0.2R
Connections:
- net GND: now also C15.1, C16.1, C18.1
- net VCC: now also C15.2, C16.2, C18.2
Other:
- moved on the sheet: D2, J1, L2
